File: PCB/v2/comms.kicad_sch (KiCad schematic)
At the start: 13 parts, among them J6 OBD, U8 TJA1051T/3, U9 TJA1027T/20

Commit message: pcb v2: lcsc numbers, availability checked
Claude-Session: https://claude.ai/code/session_015oqRiQH5gUcw5a6jvR5Zdk
Parts:
- C23, C24, C25: LCSC (none) -> C14663; MPN (none) -> CC0603KRX7R9BB104; Manufacturer (none) -> YAGEO
- D20: LCSC (none) -> C15771; MPN PESD1CAN -> PESD1CAN,215
- D21: LCSC (none) -> C148222
- J6: LCSC (none) -> C144395
- JP1, JP2: LCSC (none) -> C492401; MPN (none) -> PZ254V-11-02P; Manufacturer (none) -> XFCN
- R40: LCSC (none) -> C17909; MPN (none) -> 1206W4F1200T5E; Manufacturer (none) -> UNI-ROYAL
- R41: LCSC (none) -> C25804; MPN (none) -> 0603WAF1002T5E; Manufacturer (none) -> UNI-ROYAL
- R42: LCSC (none) -> C2934121; MPN (none) -> FRC2512J511TS; Manufacturer (none) -> FOJAN
- U8: LCSC (none) -> C58988
- U9: LCSC (none) -> C112994
Changed lines of the file:
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@@
       )
     )
-    (property "LCSC" ""
+    (property "LCSC" "C144395"
       (at 33.02 15.24 0)
       (hide yes)
@@
       )
     )
-    (property "LCSC" ""
+    (property "LCSC" "C58988"
       (at 71.12 33.02 0)
       (hide yes)
@@
       )
     )
-    (property "LCSC" ""
+    (property "LCSC" "C25804"
       (at 106.68 27.94 0)
       (hide yes)
@@
       )
     )
-    (property "MPN" ""
+    (property "MPN" "0603WAF1002T5E"
       (at 106.68 27.94 0)
       (hide yes)
@@
       )
     )
-    (property "Manufacturer" ""
+    (property "Manufacturer" "UNI-ROYAL"
       (at 106.68 27.94 0)
       (hide yes)
@@
       )
     )
-    (property "LCSC" ""
+    (property "LCSC" "C14663"
       (at 119.38 27.94 0)
       (hide yes)
@@
       )
     )
-    (property "MPN" ""
+    (property "MPN" "CC0603KRX7R9BB104"
       (at 119.38 27.94 0)
       (hide yes)
@@
       )
     )
-    (property "Manufacturer" ""
+    (property "Manufacturer" "YAGEO"
       (at 119.38 27.94 0)
       (hide yes)
@@
       )
     )
-    (property "LCSC" ""
+    (property "LCSC" "C14663"
       (at 132.08 27.94 0)
       (hide yes)
@@
       )
     )
-    (property "MPN" ""
+    (property "MPN" "CC0603KRX7R9BB104"
       (at 132.08 27.94 0)
       (hide yes)
@@
       )
     )
-    (property "Manufacturer" ""
+    (property "Manufacturer" "YAGEO"
       (at 132.08 27.94 0)
       (hide yes)
@@
       )
     )
-    (property "LCSC" ""
+    (property "LCSC" "C17909"
       (at 142.24 30.48 0)
       (hide yes)
@@
       )
     )
-    (property "MPN" ""
+    (property "MPN" "1206W4F1200T5E"
       (at 142.24 30.48 0)
       (hide yes)
@@
       )
     )
-    (property "Manufacturer" ""
+    (property "Manufacturer" "UNI-ROYAL"
       (at 142.24 30.48 0)
       (hide yes)
@@
       )
     )
-    (property "LCSC" ""
+    (property "LCSC" "C492401"
       (at 175.26 12.7 0)
       (hide yes)
@@
       )
     )
-    (property "MPN" ""
+    (property "MPN" "PZ254V-11-02P"
       (at 175.26 12.7 0)
       (hide yes)
@@
       )
     )
-    (property "Manufacturer" ""
+    (property "Manufacturer" "XFCN"
       (at 175.26 12.7 0)
       (hide yes)
@@
       )
     )
-    (property "LCSC" ""
+    (property "LCSC" "C15771"
       (at 205.74 12.7 0)
       (hide yes)
@@
       )
     )
-    (property "MPN" "PESD1CAN"
+    (property "MPN" "PESD1CAN,215"
       (at 205.74 12.7 0)
       (hide yes)
@@
       )
     )
-    (property "LCSC" ""
+    (property "LCSC" "C112994"
       (at 35.56 93.98 0)
       (hide yes)
@@
       )
     )
-    (property "LCSC" ""
+    (property "LCSC" "C14663"
       (at 71.12 88.9 0)
       (hide yes)
@@
       )
     )
-    (property "MPN" ""
+    (property "MPN" "CC0603KRX7R9BB104"
       (at 71.12 88.9 0)
       (hide yes)
@@
       )
     )
-    (property "Manufacturer" ""
+    (property "Manufacturer" "YAGEO"
       (at 71.12 88.9 0)
       (hide yes)
@@
       )
     )
-    (property "LCSC" ""
+    (property "LCSC" "C2934121"
       (at 86.36 88.9 0)
       (hide yes)
@@
       )
     )
-    (property "MPN" ""
+    (property "MPN" "FRC2512J511TS"
       (at 86.36 88.9 0)
       (hide yes)
@@
       )
     )
-    (property "Manufacturer" ""
+    (property "Manufacturer" "FOJAN"
       (at 86.36 88.9 0)
       (hide yes)
@@
       )
     )
-    (property "LCSC" ""
+    (property "LCSC" "C492401"
       (at 116.84 71.12 0)
       (hide yes)
@@
       )
     )
-    (property "MPN" ""
+    (property "MPN" "PZ254V-11-02P"
       (at 116.84 71.12 0)
       (hide yes)
@@
       )
     )
-    (property "Manufacturer" ""
+    (property "Manufacturer" "XFCN"
       (at 116.84 71.12 0)
       (hide yes)
@@
       )
     )
-    (property "LCSC" ""
+    (property "LCSC" "C148222"
       (at 144.78 71.12 0)
       (hide yes)
