File: PCB/v2/leds.kicad_sch (KiCad schematic)
At the start: 20 parts, among them J11 LED1, J12 LED2, J13 LED3, J14 LED4, J15 LED5, J16 LED6, U7 74HCT245PW

Commit message: pcb v2: lcsc numbers, availability checked
Claude-Session: https://claude.ai/code/session_015oqRiQH5gUcw5a6jvR5Zdk
Parts:
- C22: LCSC (none) -> C14663; MPN (none) -> CC0603KRX7R9BB104; Manufacturer (none) -> YAGEO
- D11, D12, D13, D14, D15, D16: LCSC (none) -> C19224; MPN PESD5V0S1BA -> PESD5V0S1BA,115
- J11, J12, J13, J14, J15, J16: LCSC (none) -> C160316
- R31, R32, R33, R34, R35, R36: LCSC (none) -> C22962; MPN (none) -> 0603WAF2200T5E; Manufacturer (none) -> UNI-ROYAL
- U7: LCSC (none) -> C5980; MPN 74HCT245PW -> 74HCT245PW,118
Changed lines of the file:
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@@
       )
     )
-    (property "LCSC" ""
+    (property "LCSC" "C5980"
       (at 40.64 43.18 0)
       (hide yes)
@@
       )
     )
-    (property "MPN" "74HCT245PW"
+    (property "MPN" "74HCT245PW,118"
       (at 40.64 43.18 0)
       (hide yes)
@@
       )
     )
-    (property "LCSC" ""
+    (property "LCSC" "C14663"
       (at 81.28 27.94 0)
       (hide yes)
@@
       )
     )
-    (property "MPN" ""
+    (property "MPN" "CC0603KRX7R9BB104"
       (at 81.28 27.94 0)
       (hide yes)
@@
       )
     )
-    (property "Manufacturer" ""
+    (property "Manufacturer" "YAGEO"
       (at 81.28 27.94 0)
       (hide yes)
@@
       )
     )
-    (property "LCSC" ""
+    (property "LCSC" "C22962"
       (at 93.98 33.02 0)
       (hide yes)
@@
       )
     )
-    (property "MPN" ""
+    (property "MPN" "0603WAF2200T5E"
       (at 93.98 33.02 0)
       (hide yes)
@@
       )
     )
-    (property "Manufacturer" ""
+    (property "Manufacturer" "UNI-ROYAL"
       (at 93.98 33.02 0)
       (hide yes)
@@
       )
     )
-    (property "LCSC" ""
+    (property "LCSC" "C19224"
       (at 124.46 12.7 0)
       (hide yes)
@@
       )
     )
-    (property "MPN" "PESD5V0S1BA"
+    (property "MPN" "PESD5V0S1BA,115"
       (at 124.46 12.7 0)
       (hide yes)
@@
       )
     )
-    (property "LCSC" ""
+    (property "LCSC" "C160316"
       (at 172.72 15.24 0)
       (hide yes)
@@
       )
     )
-    (property "LCSC" ""
+    (property "LCSC" "C22962"
       (at 182.88 33.02 0)
       (hide yes)
@@
       )
     )
-    (property "MPN" ""
+    (property "MPN" "0603WAF2200T5E"
       (at 182.88 33.02 0)
       (hide yes)
@@
       )
     )
-    (property "Manufacturer" ""
+    (property "Manufacturer" "UNI-ROYAL"
       (at 182.88 33.02 0)
       (hide yes)
@@
       )
     )
-    (property "LCSC" ""
+    (property "LCSC" "C19224"
       (at 215.9 12.7 0)
       (hide yes)
@@
       )
     )
-    (property "MPN" "PESD5V0S1BA"
+    (property "MPN" "PESD5V0S1BA,115"
       (at 215.9 12.7 0)
       (hide yes)
@@
       )
     )
-    (property "LCSC" ""
+    (property "LCSC" "C160316"
       (at 261.62 15.24 0)
       (hide yes)
@@
       )
     )
-    (property "LCSC" ""
+    (property "LCSC" "C22962"
       (at 271.78 33.02 0)
       (hide yes)
@@
       )
     )
-    (property "MPN" ""
+    (property "MPN" "0603WAF2200T5E"
       (at 271.78 33.02 0)
       (hide yes)
@@
       )
     )
-    (property "Manufacturer" ""
+    (property "Manufacturer" "UNI-ROYAL"
       (at 271.78 33.02 0)
       (hide yes)
@@
       )
     )
-    (property "LCSC" ""
+    (property "LCSC" "C19224"
       (at 35.56 91.44 0)
       (hide yes)
@@
       )
     )
-    (property "MPN" "PESD5V0S1BA"
+    (property "MPN" "PESD5V0S1BA,115"
       (at 35.56 91.44 0)
       (hide yes)
@@
       )
     )
-    (property "LCSC" ""
+    (property "LCSC" "C160316"
       (at 81.28 93.98 0)
       (hide yes)
@@
       )
     )
-    (property "LCSC" ""
+    (property "LCSC" "C22962"
       (at 93.98 111.76 0)
       (hide yes)
@@
       )
     )
-    (property "MPN" ""
+    (property "MPN" "0603WAF2200T5E"
       (at 93.98 111.76 0)
       (hide yes)
@@
       )
     )
-    (property "Manufacturer" ""
+    (property "Manufacturer" "UNI-ROYAL"
       (at 93.98 111.76 0)
       (hide yes)
@@
       )
     )
-    (property "LCSC" ""
+    (property "LCSC" "C19224"
       (at 124.46 91.44 0)
       (hide yes)
@@
       )
     )
-    (property "MPN" "PESD5V0S1BA"
+    (property "MPN" "PESD5V0S1BA,115"
       (at 124.46 91.44 0)
       (hide yes)
@@
       )
     )
-    (property "LCSC" ""
+    (property "LCSC" "C160316"
       (at 172.72 93.98 0)
       (hide yes)
@@
       )
     )
-    (property "LCSC" ""
+    (property "LCSC" "C22962"
       (at 182.88 111.76 0)
       (hide yes)
@@
       )
     )
-    (property "MPN" ""
+    (property "MPN" "0603WAF2200T5E"
       (at 182.88 111.76 0)
       (hide yes)
@@
       )
     )
-    (property "Manufacturer" ""
+    (property "Manufacturer" "UNI-ROYAL"
       (at 182.88 111.76 0)
       (hide yes)
@@
       )
     )
-    (property "LCSC" ""
+    (property "LCSC" "C19224"
       (at 213.36 91.44 0)
       (hide yes)
@@
       )
     )
-    (property "MPN" "PESD5V0S1BA"
+    (property "MPN" "PESD5V0S1BA,115"
       (at 213.36 91.44 0)
       (hide yes)
@@
       )
     )
-    (property "LCSC" ""
+    (property "LCSC" "C160316"
       (at 261.62 93.98 0)
       (hide yes)
@@
       )
     )
-    (property "LCSC" ""
+    (property "LCSC" "C22962"
       (at 271.78 111.76 0)
       (hide yes)
@@
       )
     )
-    (property "MPN" ""
+    (property "MPN" "0603WAF2200T5E"
       (at 271.78 111.76 0)
       (hide yes)
@@
       )
     )
-    (property "Manufacturer" ""
+    (property "Manufacturer" "UNI-ROYAL"
       (at 271.78 111.76 0)
       (hide yes)
@@
       )
     )
-    (property "LCSC" ""
+    (property "LCSC" "C19224"
       (at 35.56 149.86 0)
       (hide yes)
@@
       )
     )
-    (property "MPN" "PESD5V0S1BA"
+    (property "MPN" "PESD5V0S1BA,115"
       (at 35.56 149.86 0)
       (hide yes)
@@
       )
     )
-    (property "LCSC" ""
+    (property "LCSC" "C160316"
       (at 81.28 152.4 0)
       (hide yes)
