File: PCB/v2/mcu.kicad_sch (KiCad schematic)
At the start: 29 parts, among them J2 USB-C 16P, J3 UART0, J4 EXT, J5 microSD, SW1 EN, SW2 BOOT, U1 ESP32-S3-WROOM-1-N16R2, U5 LSM6DS3TR-C, U6 USBLC6-2SC6

Commit message: pcb v2: lcsc numbers, availability checked
Claude-Session: https://claude.ai/code/session_015oqRiQH5gUcw5a6jvR5Zdk
Parts:
- C16: LCSC (none) -> C45783; MPN (none) -> CL21A226MAQNNNE; Manufacturer (none) -> Samsung Electro-Mechanics
- C17, C20, C21: LCSC (none) -> C14663; MPN (none) -> CC0603KRX7R9BB104; Manufacturer (none) -> YAGEO
- C18: LCSC (none) -> C15849; MPN (none) -> CL10A105KB8NNNC; Manufacturer (none) -> Samsung Electro-Mechanics
- C19: LCSC (none) -> C15850; MPN (none) -> CL21A106KAYNNNE; Manufacturer (none) -> Samsung Electro-Mechanics
- D6: LCSC (none) -> C22371299; MPN (none) -> PSC-1608U49GC-G4; Manufacturer (none) -> HONGLITRONIC
- J3: LCSC (none) -> C2691448; MPN (none) -> PZ254V-11-04P; Manufacturer (none) -> XFCN
- J4: LCSC (none) -> C492405; MPN (none) -> PZ254V-11-06P; Manufacturer (none) -> XFCN
- J5: LCSC (none) -> C597972; MPN (none) -> DM3BT-DSF-PEJS; Manufacturer (none) -> Hirose
- R11, R12, R16, R17, R18, R19, R20, R21: LCSC (none) -> C25804; MPN (none) -> 0603WAF1002T5E; Manufacturer (none) -> UNI-ROYAL
- R13: LCSC (none) -> C21190; MPN (none) -> 0603WAF1001T5E; Manufacturer (none) -> UNI-ROYAL
- R14, R15: LCSC (none) -> C23186; MPN (none) -> 0603WAF5101T5E; Manufacturer (none) -> UNI-ROYAL
- R22, R23: LCSC (none) -> C23162; MPN (none) -> 0603WAF4701T5E; Manufacturer (none) -> UNI-ROYAL
- SW1, SW2: LCSC (none) -> C221880; MPN (none) -> PTS645SM43SMTR92LFS; Manufacturer (none) -> C&K
- U5: LCSC (none) -> C967633
- U6: LCSC (none) -> C7519
