File: PCB/v2/driftanalyser-v2.kicad_pcb (KiCad board)
At the start: 4 copper layers, 110 x 75 mm, 101 parts, among them J1 XT60PW-M, J11 LED1, J12 LED2, J13 LED3, J14 LED4, J15 LED5, J16 LED6, J2 USB-C 16P, J3 UART0, J4 EXT, J5 microSD, J6 OBD, SW1 EN, SW2 BOOT, U1 ESP32-S3-WROOM-1-N16R2, U2 BTS7002-1EPP, U3 AP63200WU-7, U4 AP7361C-33E, U5 LSM6DS3TR-C, U6 USBLC6-2SC6, U7 74HCT245PW, U8 TJA1051T/3, U9 TJA1027T/20

Commit message: pcb v2: pour the input barrel in, fixed dates in the tracked plots
Claude-Session: https://claude.ai/code/session_015oqRiQH5gUcw5a6jvR5Zdk
Routing:
- net VBAT: vias 114 -> 159

Commit message: pcb v2: link footprints to their symbols, widen the 12v arm, honest readmes
parity warnings 216 -> 18 (only the NC-pin net_conflicts left): footprints get
the library nickname, the sheet path and MPN/Manufacturer, and H1..H4 finally
have symbols. in2 12v arm now reaches U2's OUT pads - the band above them was
F.Cu only, 13.9 A, and the test only ever cut it at y=21. gerber dates fixed
inside the zip so a re-export is byte-identical, netlist source path made
relative, render-routed.svg dropped

Claude-Session: https://claude.ai/code/session_015oqRiQH5gUcw5a6jvR5Zdk
Parts:
- C1, C2: footprint CP_Elec_8x10.5 -> Capacitor_SMD:CP_Elec_8x10.5
- C10, C17, C18, C20, C21, C22, C23, C24, C25, C7, C8: footprint C_0603_1608Metric -> Capacitor_SMD:C_0603_1608Metric
- C11, C12, C13, C14, C15, C16, C19: footprint C_0805_2012Metric -> Capacitor_SMD:C_0805_2012Metric
- C3, C4, C5, C6, C9: footprint C_1210_3225Metric -> Capacitor_SMD:C_1210_3225Metric
- D1: footprint D_SMC -> Diode_SMD:D_SMC
- D11, D12, D13, D14, D15, D16: footprint D_SOD-323 -> Diode_SMD:D_SOD-323
- D2: footprint SOT-323_SC-70 -> Package_TO_SOT_SMD:SOT-323_SC-70
- D20: footprint SOT-23 -> Package_TO_SOT_SMD:SOT-23
- D21, D3, D4: footprint D_SMA -> Diode_SMD:D_SMA
- D5, D6: footprint LED_0603_1608Metric -> LED_SMD:LED_0603_1608Metric
- H1, H2, H3, H4: footprint MountingHole_3.2mm_M3 -> MountingHole:MountingHole_3.2mm_M3
- J1: footprint AMASS_XT60PW-M_1x02_P7.20mm_Horizontal -> Connector_AMASS:AMASS_XT60PW-M_1x02_P7.20mm_Horizontal
- J11, J12, J13, J14, J15, J16: footprint JST_VH_B3P-VH_1x03_P3.96mm_Vertical -> Connector_JST:JST_VH_B3P-VH_1x03_P3.96mm_Vertical
- J2: footprint USB_C_Receptacle_HRO_TYPE-C-31-M-12 -> Connector_USB:USB_C_Receptacle_HRO_TYPE-C-31-M-12
- J3: footprint PinHeader_1x04_P2.54mm_Vertical -> Connector_PinHeader_2.54mm:PinHeader_1x04_P2.54mm_Vertical
- J4: footprint PinHeader_1x06_P2.54mm_Vertical -> Connector_PinHeader_2.54mm:PinHeader_1x06_P2.54mm_Vertical
- J5: footprint microSD_HC_Hirose_DM3BT-DSF-PEJS -> Connector_Card:microSD_HC_Hirose_DM3BT-DSF-PEJS
- J6: footprint JST_XH_B4B-XH-A_1x04_P2.50mm_Vertical -> Connector_JST:JST_XH_B4B-XH-A_1x04_P2.50mm_Vertical
- JP1, JP2: footprint PinHeader_1x02_P2.54mm_Vertical -> Connector_PinHeader_2.54mm:PinHeader_1x02_P2.54mm_Vertical
- L1: footprint L_Bourns_SRN6045TA -> Inductor_SMD:L_Bourns_SRN6045TA
- R1, R10, R11, R12, R13, R14, R15, R16, R17, R18, R19, R2, R20, R21, R22, R23, R3, R31, R32, R33, R34, R35, R36, R4, R41, R5, R6, R7, R8, R9: footprint R_0603_1608Metric -> Resistor_SMD:R_0603_1608Metric
- R40: footprint R_1206_3216Metric -> Resistor_SMD:R_1206_3216Metric
- R42: footprint R_2512_6332Metric -> Resistor_SMD:R_2512_6332Metric
- SW1, SW2: footprint SW_SPST_PTS645Sx43SMTR92 -> Button_Switch_SMD:SW_SPST_PTS645Sx43SMTR92
- U1: footprint ESP32-S3-WROOM-1 -> RF_Module:ESP32-S3-WROOM-1
- U2: footprint PG-TSDSO-14 -> da2:PG-TSDSO-14
- U3: footprint TSOT-23-6 -> Package_TO_SOT_SMD:TSOT-23-6
- U4: footprint SOT-223-3_TabPin2 -> Package_TO_SOT_SMD:SOT-223-3_TabPin2
- U5: footprint LGA-14_3x2.5mm_P0.5mm_LayoutBorder3x4y -> Package_LGA:LGA-14_3x2.5mm_P0.5mm_LayoutBorder3x4y
- U6: footprint SOT-23-6 -> Package_TO_SOT_SMD:SOT-23-6
- U7: footprint TSSOP-20_4.4x6.5mm_P0.65mm -> Package_SO:TSSOP-20_4.4x6.5mm_P0.65mm
- U8, U9: footprint SOIC-8_3.9x4.9mm_P1.27mm -> Package_SO:SOIC-8_3.9x4.9mm_P1.27mm

Commit message: pcb v2: c1/c2 are 50v not 35v
GVZ1H107M0810CNVC (C2983550) is a 50V part, the 35V label was a typo. same part, nothing to reorder

Claude-Session: https://claude.ai/code/session_011XKWp7yoGtzw88WQygPeEA
Parts:
- C1, C2: value 100uF 35V -> 100uF 50V
Changed lines of the file:
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@@
 			)
 		)
-		(property "Value" "100uF 35V"
+		(property "Value" "100uF 50V"
 			(at 0 5.3 0)
 			(layer "F.Fab")
@@
 			)
 		)
-		(property "Value" "100uF 35V"
+		(property "Value" "100uF 50V"
 			(at 0 5.3 0)
 			(layer "F.Fab")
