File: PCB/v3/mcu.kicad_sch (KiCad schematic)
At the start: 19 parts, among them J3 USB-C 16P, J4 UART0, SW1 BOOT, SW2 EN, U1 ESP32-S3-WROOM-1U-N16R2, U3 LSM6DS3TR-C, U9 USBLC6-2SC6

Commit message: pcb v3: lcsc numbers, lmr36520 buck
ap63200 vin abs max was under the smcj24ca clamp, j2 stud hand-fit
Parts:
- U1: LCSC (none) -> C3013945
Changed lines of the file:
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@@
+      )
+    )
+    (property "LCSC" "C3013945"
+      (at 48.26 53.34 0)
+      (hide yes)
+      (effects
+        (font
+          (size 1.27 1.27)
+        )
       )
     )
