File: PCB/v3/outputs.kicad_sch (KiCad schematic)
At the start: 74 parts, among them U10 BTS7008-2EPA, U11 BTS7008-2EPA, U12 BTS7008-2EPA, U13 BTS7008-2EPA, U14 PCA9555PW, U15 74HCT245PW, U16 74HCT245PW

Commit message: pcb v3: lcsc numbers, lmr36520 buck
ap63200 vin abs max was under the smcj24ca clamp, j2 stud hand-fit
Parts:
- C21, C22, C24, C25, C27, C28, C30, C31, C32: MPN CL10B103KB8NNNC -> 0603B103K500NT; Manufacturer Samsung Electro-Mechanics -> FH
- D10: LCSC (none) -> C47546; MPN BAT54S -> BAT54S,215
- U10, U11, U12, U13: LCSC (none) -> C534830; MPN BTS70082EPAXUMA1 -> BTS7008-2EPA
- U14: LCSC (none) -> C128392
Changed lines of the file:
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@@
       )
     )
-    (property "MPN" "BTS70082EPAXUMA1"
+    (property "LCSC" "C534830"
+      (at 238.76 22.86 0)
+      (hide yes)
+      (effects
+        (font
+          (size 1.27 1.27)
+        )
+      )
+    )
+    (property "MPN" "BTS7008-2EPA"
       (at 238.76 22.86 0)
       (hide yes)
@@
       )
     )
-    (property "MPN" "CL10B103KB8NNNC"
+    (property "MPN" "0603B103K500NT"
       (at 325.12 33.02 0)
       (hide yes)
@@
       )
     )
-    (property "Manufacturer" "Samsung Electro-Mechanics"
+    (property "Manufacturer" "FH"
       (at 325.12 33.02 0)
       (hide yes)
@@
       )
     )
-    (property "MPN" "CL10B103KB8NNNC"
+    (property "MPN" "0603B103K500NT"
       (at 340.36 33.02 0)
       (hide yes)
@@
       )
     )
-    (property "Manufacturer" "Samsung Electro-Mechanics"
+    (property "Manufacturer" "FH"
       (at 340.36 33.02 0)
       (hide yes)
@@
       )
     )
-    (property "MPN" "BTS70082EPAXUMA1"
+    (property "LCSC" "C534830"
+      (at 386.08 22.86 0)
+      (hide yes)
+      (effects
+        (font
+          (size 1.27 1.27)
+        )
+      )
+    )
+    (property "MPN" "BTS7008-2EPA"
       (at 386.08 22.86 0)
       (hide yes)
@@
       )
     )
-    (property "MPN" "CL10B103KB8NNNC"
+    (property "MPN" "0603B103K500NT"
       (at 472.44 33.02 0)
       (hide yes)
@@
       )
     )
-    (property "Manufacturer" "Samsung Electro-Mechanics"
+    (property "Manufacturer" "FH"
       (at 472.44 33.02 0)
       (hide yes)
@@
       )
     )
-    (property "MPN" "CL10B103KB8NNNC"
+    (property "MPN" "0603B103K500NT"
       (at 490.22 33.02 0)
       (hide yes)
@@
       )
     )
-    (property "Manufacturer" "Samsung Electro-Mechanics"
+    (property "Manufacturer" "FH"
       (at 490.22 33.02 0)
       (hide yes)
@@
       )
     )
-    (property "MPN" "BTS70082EPAXUMA1"
+    (property "LCSC" "C534830"
+      (at 535.94 22.86 0)
+      (hide yes)
+      (effects
+        (font
+          (size 1.27 1.27)
+        )
+      )
+    )
+    (property "MPN" "BTS7008-2EPA"
       (at 535.94 22.86 0)
       (hide yes)
@@
       )
     )
-    (property "MPN" "CL10B103KB8NNNC"
+    (property "MPN" "0603B103K500NT"
       (at 53.34 91.44 0)
       (hide yes)
@@
       )
     )
-    (property "Manufacturer" "Samsung Electro-Mechanics"
+    (property "Manufacturer" "FH"
       (at 53.34 91.44 0)
       (hide yes)
@@
       )
     )
-    (property "MPN" "CL10B103KB8NNNC"
+    (property "MPN" "0603B103K500NT"
       (at 68.58 91.44 0)
       (hide yes)
@@
       )
     )
-    (property "Manufacturer" "Samsung Electro-Mechanics"
+    (property "Manufacturer" "FH"
       (at 68.58 91.44 0)
       (hide yes)
@@
       )
     )
-    (property "MPN" "BTS70082EPAXUMA1"
+    (property "LCSC" "C534830"
+      (at 114.3 81.28 0)
+      (hide yes)
+      (effects
+        (font
+          (size 1.27 1.27)
+        )
+      )
+    )
+    (property "MPN" "BTS7008-2EPA"
       (at 114.3 81.28 0)
       (hide yes)
@@
       )
     )
-    (property "MPN" "CL10B103KB8NNNC"
+    (property "MPN" "0603B103K500NT"
       (at 200.66 91.44 0)
       (hide yes)
@@
       )
     )
-    (property "Manufacturer" "Samsung Electro-Mechanics"
+    (property "Manufacturer" "FH"
       (at 200.66 91.44 0)
       (hide yes)
@@
       )
     )
-    (property "MPN" "CL10B103KB8NNNC"
+    (property "MPN" "0603B103K500NT"
       (at 218.44 91.44 0)
       (hide yes)
@@
       )
     )
-    (property "Manufacturer" "Samsung Electro-Mechanics"
+    (property "Manufacturer" "FH"
       (at 218.44 91.44 0)
       (hide yes)
@@
       )
     )
-    (property "MPN" "CL10B103KB8NNNC"
+    (property "MPN" "0603B103K500NT"
       (at 256.54 93.98 0)
       (hide yes)
@@
       )
     )
-    (property "Manufacturer" "Samsung Electro-Mechanics"
+    (property "Manufacturer" "FH"
       (at 256.54 93.98 0)
       (hide yes)
@@
       )
     )
-    (property "MPN" "BAT54S"
+    (property "LCSC" "C47546"
+      (at 284.48 71.12 0)
+      (hide yes)
+      (effects
+        (font
+          (size 1.27 1.27)
+        )
+      )
+    )
+    (property "MPN" "BAT54S,215"
       (at 284.48 71.12 0)
       (hide yes)
@@
       (at 342.9 106.68 0)
       (hide yes)
+      (effects
+        (font
+          (size 1.27 1.27)
+        )
+      )
+    )
+    (property "LCSC" "C128392"
+      (at 342.9 106.68 0)
+      (hide yes)
