File: PCB/v3/driftanalyser-v3.kicad_pcb (KiCad board)
At the start: 6 copper layers, 55 x 112 mm, 173 parts, among them J1 6437288-1, J2 Stud_M6, J3 USB-C 16P, J4 UART0, J5 Stud_M6, Q1 BSC016N06NS, Q2 BSC016N06NS, SW1 BOOT, SW2 EN, U1 ESP32-S3-WROOM-1U-N16R2, U10 BTS7008-2EPA, U11 BTS7008-2EPA, U12 BTS7008-2EPA, U13 BTS7008-2EPA, U14 PCA9555PW, U15 74HCT245PW, U16 74HCT245PW, U2 LM74700-Q1, U3 LSM6DS3TR-C, U4 TJA1051T/3, U5 TJA1027T/20, U6 TPS2553DBV, U7 LMR36520ADDAR, U8 AP7361C-33E, U9 USBLC6-2SC6

Commit message: pcb v3: j5 seam vias, boot silk off u9
vias on the disc edge so the j5 disc and the gnd fill share copper, not just an edge

Claude-Session: https://claude.ai/code/session_01MELKvCtSrN4XHin3AfxGm6
Routing:
- net GND: vias 144 -> 173
Changed lines of the file:
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@@
 	)
 	(gr_text "BOOT"
-		(at 23.9 103 90)
+		(at 24 103.9 90)
 		(layer "F.SilkS")
 		(effects
@@
 	)
 	(via
+		(at 38.722 104.41)
+		(size 0.8)
+		(drill 0.4)
+		(layers "F.Cu" "B.Cu")
+		(net "GND")
+	)
+	(via
 		(at 35.241 94.685)
 		(size 0.8)
@@
 	)
 	(via
+		(at 51.4 103.3)
+		(size 0.8)
+		(drill 0.4)
+		(layers "F.Cu" "B.Cu")
+		(net "GND")
+	)
+	(via
+		(at 40.216 105.272)
+		(size 0.8)
+		(drill 0.4)
+		(layers "F.Cu" "B.Cu")
+		(net "GND")
+	)
+	(via
 		(at 32 61.425)
 		(size 0.6)
@@
 	)
 	(via
+		(at 34.837 93.738)
+		(size 0.8)
+		(drill 0.4)
+		(layers "F.Cu" "B.Cu")
+		(net "GND")
+	)
+	(via
+		(at 36.29 101.978)
+		(size 0.8)
+		(drill 0.4)
+		(layers "F.Cu" "B.Cu")
+		(net "GND")
+	)
+	(via
 		(at 47.581 105.039)
 		(size 0.8)
@@
 	)
 	(via
+		(at 35.428 92.116)
+		(size 0.8)
+		(drill 0.4)
+		(layers "F.Cu" "B.Cu")
+		(net "GND")
+	)
+	(via
 		(at 44.2 68.025)
 		(size 0.6)
@@
 	)
 	(via
+		(at 46.962 86.737)
+		(size 0.8)
+		(drill 0.4)
+		(layers "F.Cu" "B.Cu")
+		(net "GND")
+	)
+	(via
 		(at 18.15 102.23)
 		(size 0.6)
@@
 	)
 	(via
+		(at 50.078 104.41)
+		(size 0.8)
+		(drill 0.4)
+		(layers "F.Cu" "B.Cu")
+		(net "GND")
+	)
+	(via
 		(at 15.225 43.125)
 		(size 0.6)
@@
 	)
 	(via
+		(at 45.263 106.162)
+		(size 0.8)
+		(drill 0.4)
+		(layers "F.Cu" "B.Cu")
+		(net "GND")
+	)
+	(via
 		(at 13.075 36.725)
 		(size 0.6)
@@
 	)
 	(via
+		(at 40.216 87.328)
+		(size 0.8)
+		(drill 0.4)
+		(layers "F.Cu" "B.Cu")
+		(net "GND")
+	)
+	(via
 		(at 30 95.875)
 		(size 0.6)
@@
 	)
 	(via
+		(at 51.4 89.3)
+		(size 0.8)
+		(drill 0.4)
+		(layers "F.Cu" "B.Cu")
+		(net "GND")
+	)
+	(via
 		(at 37.276 90.322)
 		(size 0.8)
@@
 	)
 	(via
+		(at 52.51 90.622)
+		(size 0.8)
+		(drill 0.4)
+		(layers "F.Cu" "B.Cu")
+		(net "GND")
+	)
+	(via
 		(at 41.875 82.855)
 		(size 0.6)
@@
 	)
 	(via
+		(at 37.4 103.3)
+		(size 0.8)
+		(drill 0.4)
+		(layers "F.Cu" "B.Cu")
+		(net "GND")
+	)
+	(via
+		(at 52.51 101.978)
+		(size 0.8)
+		(drill 0.4)
+		(layers "F.Cu" "B.Cu")
+		(net "GND")
+	)
+	(via
+		(at 35.428 100.484)
+		(size 0.8)
+		(drill 0.4)
+		(layers "F.Cu" "B.Cu")
+		(net "GND")
+	)
+	(via
+		(at 53.963 93.738)
+		(size 0.8)
+		(drill 0.4)
+		(layers "F.Cu" "B.Cu")
+		(net "GND")
+	)
+	(via
+		(at 53.372 92.116)
+		(size 0.8)
+		(drill 0.4)
+		(layers "F.Cu" "B.Cu")
+		(net "GND")
+	)
+	(via
 		(at 26.075 36.025)
 		(size 0.6)
@@
 	)
 	(via
+		(at 48.584 87.328)
+		(size 0.8)
+		(drill 0.4)
+		(layers "F.Cu" "B.Cu")
+		(net "GND")
+	)
+	(via
 		(at 25.4 65.225)
 		(size 0.6)
@@
 	)
 	(via
+		(at 36.29 90.622)
+		(size 0.8)
+		(drill 0.4)
+		(layers "F.Cu" "B.Cu")
+		(net "GND")
+	)
+	(via
+		(at 37.4 89.3)
+		(size 0.8)
+		(drill 0.4)
+		(layers "F.Cu" "B.Cu")
+		(net "GND")
+	)
+	(via
 		(at 41.875 36.725)
 		(size 0.6)
@@
 	)
 	(via
+		(at 48.584 105.272)
+		(size 0.8)
+		(drill 0.4)
+		(layers "F.Cu" "B.Cu")
+		(net "GND")
+	)
+	(via
 		(at 45.9 68.025)
 		(size 0.6)
@@
 	)
 	(via
+		(at 53.963 98.862)
+		(size 0.8)
+		(drill 0.4)
+		(layers "F.Cu" "B.Cu")
+		(net "GND")
+	)
+	(via
 		(at 32.4 85.625)
 		(size 0.6)
@@
 	)
 	(via
+		(at 46.962 105.863)
+		(size 0.8)
+		(drill 0.4)
+		(layers "F.Cu" "B.Cu")
+		(net "GND")
+	)
+	(via
 		(at 49.05 104.354)
 		(size 0.8)
@@
 	)
 	(via
+		(at 34.837 98.862)
+		(size 0.8)
+		(drill 0.4)
+		(layers "F.Cu" "B.Cu")
+		(net "GND")
+	)
+	(via
 		(at 35.241 97.915)
 		(size 0.8)
@@
 	)
 	(via
+		(at 50.078 88.19)
+		(size 0.8)
+		(drill 0.4)
+		(layers "F.Cu" "B.Cu")
+		(net "GND")
+	)
+	(via
 		(at 36.05 40.575)
 		(size 0.6)
@@
 	)
 	(via
+		(at 38.722 88.19)
+		(size 0.8)
+		(drill 0.4)
+		(layers "F.Cu" "B.Cu")
+		(net "GND")
+	)
+	(via
 		(at 44.2 78.325)
 		(size 0.6)
@@
 	)
 	(via
+		(at 43.537 106.162)
+		(size 0.8)
+		(drill 0.4)
+		(layers "F.Cu" "B.Cu")
+		(net "GND")
+	)
+	(via
 		(at 25.62 81.25)
 		(size 0.6)
@@
 	)
 	(via
+		(at 53.372 100.484)
+		(size 0.8)
+		(drill 0.4)
+		(layers "F.Cu" "B.Cu")
+		(net "GND")
+	)
+	(via
 		(at 22.2 74.9)
 		(size 0.6)
@@
 		(layers "F.Cu" "B.Cu")
 		(net "GND")
+	)
+	(via
+		(at 41.838 105.863)
+		(size 0.8)
+		(drill 0.4)
+		(layers "F.Cu" "B.Cu")
+		(net "GND")

Commit message: pcb v3: real redcube footprint for the studs
16 press-fit pins per the wurth 7461059 drawing, j5 via ring off the body

Claude-Session: https://claude.ai/code/session_01MELKvCtSrN4XHin3AfxGm6
Parts:
- J2, J5: value Stud_M6 -> 7461059 M6; footprint da3:Stud_M6 -> da3:Wurth_REDCUBE_7461059
Routing:
- net VIN: vias 82 -> 78
- added copper zone on B.Cu, net VIN
- added copper zone on In1.Cu, net VIN
- added copper zone on In2.Cu, net VIN
- added copper zone on In4.Cu, net VIN
