File: PCB/v3/driftanalyser-v3.kicad_pcb (KiCad board)
At the start: 6 copper layers, 55 x 112 mm, 173 parts, among them J1 6437288-1, J2 7461059 M6, J3 USB-C 16P, J4 UART0, J5 7461059 M6, Q1 BSC016N06NS, Q2 BSC016N06NS, SW1 BOOT, SW2 EN, U1 ESP32-S3-WROOM-1U-N16R2, U10 BTS7008-2EPA, U11 BTS7008-2EPA, U12 BTS7008-2EPA, U13 BTS7008-2EPA, U14 PCA9555PW, U15 74HCT245PW, U16 74HCT245PW, U2 LM74700-Q1, U3 LSM6DS3TR-C, U4 TJA1051T/3, U5 TJA1027T/20, U6 TPS2553DBV, U7 LMR36520ADDAR, U8 AP7361C-33E, U9 USBLC6-2SC6

Commit message: pcb v3: vbat divider 470k/100k, r19 100k, r8 10k
Claude-Session: https://claude.ai/code/session_01MELKvCtSrN4XHin3AfxGm6
Parts:
- R1: value 47k -> 470k
- R19, R2: value 10k -> 100k
- R8: value 100k -> 10k
Changed lines of the file:
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@@
 			)
 		)
-		(property "Value" "10k"
+		(property "Value" "100k"
 			(at 0 1.43 90)
 			(layer "F.Fab")
@@
 			)
 		)
-		(property "LCSC" "C25804"
+		(property "LCSC" "C25803"
 			(at 0 0 90)
 			(layer "F.Fab")
@@
 			)
 		)
-		(property "MPN" "0603WAF1002T5E"
+		(property "MPN" "0603WAF1003T5E"
 			(at 0 0 90)
 			(layer "F.Fab")
@@
 			)
 		)
-		(property "Value" "10k"
+		(property "Value" "100k"
 			(at 0 1.43 90)
 			(layer "F.Fab")
@@
 			)
 		)
-		(property "LCSC" "C25804"
+		(property "LCSC" "C25803"
 			(at 0 0 90)
 			(layer "F.Fab")
@@
 			)
 		)
-		(property "MPN" "0603WAF1002T5E"
+		(property "MPN" "0603WAF1003T5E"
 			(at 0 0 90)
 			(layer "F.Fab")
@@
 			)
 		)
-		(property "Value" "47k"
+		(property "Value" "470k"
 			(at 0 1.43 90)
 			(layer "F.Fab")
@@
 			)
 		)
-		(property "LCSC" "C25819"
+		(property "LCSC" "C23178"
 			(at 0 0 90)
 			(layer "F.Fab")
@@
 			)
 		)
-		(property "MPN" "0603WAF4702T5E"
+		(property "MPN" "0603WAF4703T5E"
 			(at 0 0 90)
 			(layer "F.Fab")
@@
 			)
 		)
-		(property "Value" "100k"
+		(property "Value" "10k"
 			(at 0 1.43 90)
 			(layer "F.Fab")
@@
 			)
 		)
-		(property "LCSC" "C25803"
+		(property "LCSC" "C25804"
 			(at 0 0 90)
 			(layer "F.Fab")
@@
 			)
 		)
-		(property "MPN" "0603WAF1003T5E"
+		(property "MPN" "0603WAF1002T5E"
 			(at 0 0 90)
 			(layer "F.Fab")

Commit message: pcb v3: q1/q2 lead pads per infineon fl land
Claude-Session: https://claude.ai/code/session_01MELKvCtSrN4XHin3AfxGm6
Parts:
- Q1, Q2: footprint Package_TO_SOT_SMD:TDSON-8-1 -> da3:Infineon_TDSON-8_FL
