File: PCB/v3/power.kicad_sch (KiCad schematic)
At the start: 47 parts, among them J2 Stud_M6, Q1 BSC016N06NS, Q2 BSC016N06NS, U2 LM74700-Q1, U6 TPS2553DBV, U7 AP63200WU-7, U8 AP7361C-33E

Commit message: pcb v3: lcsc numbers, lmr36520 buck
ap63200 vin abs max was under the smcj24ca clamp, j2 stud hand-fit
Parts:
- added C37: 220nF 100V, Capacitor_SMD:C_0805_2012Metric, symbol Device:C
- added C38: 1uF, Capacitor_SMD:C_0603_1608Metric, symbol Device:C
- added R19: 10k, Resistor_SMD:R_0603_1608Metric, symbol Device:R
- C2: LCSC (none) -> C21120; MPN (none) -> CL10B224KA8NNNC; Manufacturer (none) -> Samsung Electro-Mechanics
- D1: LCSC (none) -> C151279
- D2, D3: LCSC (none) -> C47546; MPN BAT54S -> BAT54S,215
- J2: MPN 7461059 -> 7461059 (hand-fit)
- L1: value 6.8uH -> 10uH; LCSC C341066 -> C2046332; MPN YNR6045-6R8M -> SRN6045TA-100M; Manufacturer YJYCOIN -> Bourns
- Q1, Q2: LCSC (none) -> C454269; MPN BSC016N06NSATMA1 -> BSC016N06NS
- R10: value 10k -> 22.6k; LCSC C25804 -> C100874; MPN 0603WAF1002T5E -> CR0603FA2262G; Manufacturer UNI-ROYAL -> LIZ Elec
- R11: LCSC (none) -> C22952; MPN (none) -> 0603WAF2103T5E; Manufacturer (none) -> UNI-ROYAL
- R6: LCSC (none) -> C4216; MPN (none) -> 0603WAF3302T5E; Manufacturer (none) -> UNI-ROYAL
- R9: value 57.6k -> 100k; LCSC C2933240 -> C25803; MPN FRC0603F5762TS -> 0603WAF1003T5E; Manufacturer FOJAN -> UNI-ROYAL
- U2: LCSC (none) -> C3236229
- U6: LCSC (none) -> C55266
- U7: value AP63200WU-7 -> LMR36520ADDAR; footprint Package_TO_SOT_SMD:TSOT-23-6 -> Package_SO:Texas_HTSOP-8-1EP_3.9x4.9mm_P1.27mm_EP2.95x4.9mm_Mask2.4x3.1mm_ThermalVias; symbol Regulator_Switching:AP63200WU -> da3:LMR36520ADDA; LCSC C2071868 -> C2879422; MPN AP63200WU-7 -> LMR36520ADDAR; Manufacturer Diodes Incorporated -> Texas Instruments
Connections:
- net BUCK_BST: now also U7.7 (BOOT); no longer U7.6 (BST)
- net BUCK_FB: now also U7.5 (FB); no longer U7.1 (FB)
- net BUCK_SW: now also U7.8 (SW); no longer U7.5 (SW)
- net GND: now also U7.1 (PGND), U7.9 (PAD), C37.2, C38.2; no longer U7.4 (GND)
- net PWR_EN: now also R19.1; no longer U7.2 (EN)
- net VBUS: now also U7.2 (VIN), C37.1; no longer U7.3 (IN)
- new net BUCK_EN: R19.2, U7.3 (EN)
- new net BUCK_VCC: C38.1, U7.6 (VCC)
- no-connect marks 4 -> 5
Other:
- moved on the sheet: C10, C11, C12, C13, C14, C15, C7, C8, C9, D6, D7, H1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

Commit message: pcb v3: gnd stud j5, board 55x112 (placement only)
doesnt fit in 100, unrouted, needs author ok on the size
Claude-Session: https://claude.ai/code/session_01MELKvCtSrN4XHin3AfxGm6
Parts:
- added J5: Stud_M6, da3:Stud_M6, symbol Connector_Generic:Conn_01x01
Connections:
- net GND: now also J5.1 (Pin_1)
Other:
- moved on the sheet: C1, C2, C3, C4, C5, C6, D1, D2, Q1, Q2, R1, R2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

Commit message: pcb v3: real redcube footprint for the studs
16 press-fit pins per the wurth 7461059 drawing, j5 via ring off the body

Claude-Session: https://claude.ai/code/session_01MELKvCtSrN4XHin3AfxGm6
Parts:
- J2, J5: value Stud_M6 -> 7461059 M6; footprint da3:Stud_M6 -> da3:Wurth_REDCUBE_7461059
Changed lines of the file:
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@@
       )
     )
-    (property "Value" "Stud_M6"
+    (property "Value" "7461059 M6"
       (at 22.46 19.47 0)
       (effects
@@
       )
     )
-    (property "Footprint" "da3:Stud_M6"
+    (property "Footprint" "da3:Wurth_REDCUBE_7461059"
       (at 30.48 12.7 0)
       (hide yes)
@@
       )
     )
-    (property "Value" "Stud_M6"
+    (property "Value" "7461059 M6"
       (at 47.86 19.47 0)
       (effects
@@
       )
     )
-    (property "Footprint" "da3:Stud_M6"
+    (property "Footprint" "da3:Wurth_REDCUBE_7461059"
       (at 55.88 12.7 0)
       (hide yes)

Commit message: pcb v3: vbat divider 470k/100k, r19 100k, r8 10k
Claude-Session: https://claude.ai/code/session_01MELKvCtSrN4XHin3AfxGm6
Parts:
- R1: value 47k -> 470k; LCSC C25819 -> C23178; MPN 0603WAF4702T5E -> 0603WAF4703T5E
- R19, R2: value 10k -> 100k; LCSC C25804 -> C25803; MPN 0603WAF1002T5E -> 0603WAF1003T5E
- R8: value 100k -> 10k; LCSC C25803 -> C25804; MPN 0603WAF1003T5E -> 0603WAF1002T5E
Other:
- moved on the sheet: C6, D2, R2, R3

Commit message: pcb v3: q1/q2 lead pads per infineon fl land
Claude-Session: https://claude.ai/code/session_01MELKvCtSrN4XHin3AfxGm6
Parts:
- Q1, Q2: footprint Package_TO_SOT_SMD:TDSON-8-1 -> da3:Infineon_TDSON-8_FL
Changed lines of the file:
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@@
       )
     )
-    (property "Footprint" "Package_TO_SOT_SMD:TDSON-8-1"
+    (property "Footprint" "da3:Infineon_TDSON-8_FL"
       (at 215.9 30.48 0)
       (hide yes)
@@
       )
     )
-    (property "Footprint" "Package_TO_SOT_SMD:TDSON-8-1"
+    (property "Footprint" "da3:Infineon_TDSON-8_FL"
       (at 248.92 30.48 0)
       (hide yes)
